Commit message: arm's links visual material changed

File: owr_description/urdf/owr.urdf.xacro (robot description, xacro)
@@ -95,6 +95,6 @@
                     <mesh filename="${bl_dae}"/>
                 </geometry>
-                <material name="">
-                    <color rgba="0.439216 0.47451 0.501961 1.0" />
+                <material name="LightGrey">
+                    <color rgba="0.7 0.7 0.7 1.0"/>
                 </material>
             </visual>
@@ -130,6 +130,6 @@
                     <mesh filename="${bsl_dae}"/>
                 </geometry> -->
-                <material name="">
-                    <color rgba="0.866667 0.321569 0.156863 1.0" />
+                <material name="LightGrey">
+                    <color rgba="0.7 0.7 0.7 1.0"/>
                 </material>
             </visual>
@@ -165,6 +165,6 @@
                     <mesh filename="${sel_stl}" />
                 </geometry>
-                <material name="">
-                    <color rgba="1 0.756863 0.054902 1.0" />
+                <material name="LightGrey">
+                    <color rgba="0.7 0.7 0.7 1.0"/>
                 </material>
             </visual>
@@ -200,6 +200,6 @@
                     <mesh filename="${ew1l_stl}" />
                 </geometry>
-                <material name="">
-                    <color rgba="0.372549 0.654902 0.239216 1.0" />
+                <material name="LightGrey">
+                    <color rgba="0.7 0.7 0.7 1.0"/>
                 </material>
             </visual>
@@ -235,6 +235,6 @@
                     <mesh filename="${w1w2l_stl}" />
                 </geometry>
-                <material name="">
-                    <color rgba="0.32549 0.529412 0.752941 1.0" />
+                <material name="LightGrey">
+                    <color rgba="0.7 0.7 0.7 1.0"/>
                 </material>
             </visual>
@@ -270,6 +270,6 @@
                     <mesh filename="${w2w3l_stl}" />
                 </geometry>
-                <material name="">
-                    <color rgba="0.513725 0.415686 0.733333 1.0" />
+                <material name="LightGrey">
+                    <color rgba="0.7 0.7 0.7 1.0"/>
                 </material>
             </visual>
@@ -305,6 +305,6 @@
                     <mesh filename="${w3eefl_stl}" />
                 </geometry>
-                <material name="">
-                    <color rgba="0.901961 0.901961 0.901961 1.0" />
+                <material name="LightGrey">
+                    <color rgba="0.7 0.7 0.7 1.0"/>
                 </material>
             </visual>
