Commit message: owr_EEF_Link_gripper_base origin set to x=0

File: owr_description/urdf/gripper/owr_robotiq_140.xacro (robot description, xacro)
@@ -25,5 +25,5 @@
       <!--force torque sensor-->
       <xacro:robotiq_fts150 prefix="" parent="EEF_Link" >
-        <origin xyz="0.009 0 0 " rpy="-${pi/2} 0 -${pi/2}"/>
+        <origin xyz="0 0 0 " rpy="-${pi/2} 0 -${pi/2}"/>
       </xacro:robotiq_fts150>
       <!-- gripper -->
@@ -32,5 +32,5 @@
         <parent link= "${prefix}fts_toolside" />
         <child link = "${prefix}robotiq_arg2f_base_link" />
-        <origin xyz=" 0.0 0.0 0.0" rpy="0.0 0.0 ${pi/2}" />
+        <origin xyz="0 0 0" rpy="0 0 ${pi/2}" />
       </joint>
       <!--<link name="${prefix}tool" />
