Commit message: link visual material changed for gazebo

File: owr_description/urdf/gripper/robotiq_arg2f.xacro (robot description, xacro)
@@ -24,6 +24,7 @@
       </collision>
     </link>
-    <!--<gazebo reference="${prefix}robotiq_arg2f_base_link">
-      <selfCollide>true</selfCollide>
+    <gazebo reference="${prefix}robotiq_arg2f_base_link">
+      <material>Gazebo/Grey</material>
+     <!-- <selfCollide>true</selfCollide>
       <gravity>false</gravity>
       <implicitSpringDamper>1</implicitSpringDamper>
@@ -31,6 +32,6 @@
       <mu2>100000</mu2>
       <kp>100000000.0</kp>
-      <kd>1.0</kd>
-    </gazebo>-->
+      <kd>1.0</kd>-->
+    </gazebo>
   </xacro:macro>
   <xacro:macro name="finger_joints" params="prefix fingerprefix reflect">

File: owr_description/urdf/gripper/robotiq_arg2f_140_model_macro.xacro (robot description, xacro)
@@ -31,14 +31,15 @@
       </collision>
     </link>
-    <!--<gazebo reference="${prefix}${fingerprefix}_outer_knuckle">
-      <selfCollide>true</selfCollide>
-      <gravity>false</gravity>
-      <implicitSpringDamper>1</implicitSpringDamper>
-      <mu1>100000</mu1>
-      <mu2>100000</mu2>
-      <kp>100000000.0</kp>
-      <kd>1.0</kd>
-      <maxVel>0</maxVel>
-    </gazebo>-->
+    <gazebo reference="${prefix}${fingerprefix}_outer_knuckle">
+      <material>Gazebo/Black</material>
+      <!--<selfCollide>true</selfCollide>
+      <gravity>false</gravity>
+      <implicitSpringDamper>1</implicitSpringDamper>
+      <mu1>100000</mu1>
+      <mu2>100000</mu2>
+      <kp>100000000.0</kp>
+      <kd>1.0</kd>
+      <maxVel>0</maxVel>-->
+    </gazebo>
   </xacro:macro>
   <xacro:macro name="outer_finger" params="prefix fingerprefix stroke">
@@ -71,13 +72,15 @@
       </collision>
     </link>
-    <!--<gazebo reference="${prefix}${fingerprefix}_outer_finger">
-      <selfCollide>true</selfCollide>
-      <gravity>false</gravity>
-      <implicitSpringDamper>1</implicitSpringDamper>
-      <mu1>100000</mu1>
-      <mu2>100000</mu2>
-      <kp>100000000.0</kp>
-      <kd>1.0</kd>
-    </gazebo>-->
+    <gazebo reference="${prefix}${fingerprefix}_outer_finger">
+      <material>Gazebo/Black</material>
+      <!--<selfCollide>true</selfCollide>
+      <gravity>false</gravity>
+      <implicitSpringDamper>1</implicitSpringDamper>
+      <mu1>100000</mu1>
+      <mu2>100000</mu2>
+      <kp>100000000.0</kp>
+      <kd>1.0</kd>
+      <maxVel>0</maxVel>-->
+    </gazebo>
   </xacro:macro>
   <xacro:macro name="inner_knuckle" params="prefix fingerprefix stroke">
@@ -110,13 +113,15 @@
       </collision>
     </link>
-    <!--<gazebo reference="${prefix}${fingerprefix}_inner_knuckle">
-      <selfCollide>true</selfCollide>
-      <gravity>false</gravity>
-      <implicitSpringDamper>1</implicitSpringDamper>
-      <mu1>100000</mu1>
-      <mu2>100000</mu2>
-      <kp>100000000.0</kp>
-      <kd>1.0</kd>
-    </gazebo>-->
+    <gazebo reference="${prefix}${fingerprefix}_inner_knuckle">
+      <material>Gazebo/Black</material>
+      <!--<selfCollide>true</selfCollide>
+      <gravity>false</gravity>
+      <implicitSpringDamper>1</implicitSpringDamper>
+      <mu1>100000</mu1>
+      <mu2>100000</mu2>
+      <kp>100000000.0</kp>
+      <kd>1.0</kd>
+      <maxVel>0</maxVel>-->
+    </gazebo>
   </xacro:macro>
   <xacro:macro name="inner_finger" params="prefix fingerprefix stroke">
@@ -149,13 +154,15 @@
       </collision>
     </link>
-    <!--<gazebo reference="${prefix}${fingerprefix}_inner_finger">
-      <selfCollide>true</selfCollide>
-      <gravity>false</gravity>
-      <implicitSpringDamper>1</implicitSpringDamper>
-      <mu1>100000</mu1>
-      <mu2>100000</mu2>
-      <kp>100000000.0</kp>
-      <kd>1.0</kd>
-    </gazebo>-->
+    <gazebo reference="${prefix}${fingerprefix}_inner_finger">
+      <material>Gazebo/Black</material>
+      <!--<selfCollide>true</selfCollide>
+      <gravity>false</gravity>
+      <implicitSpringDamper>1</implicitSpringDamper>
+      <mu1>100000</mu1>
+      <mu2>100000</mu2>
+      <kp>100000000.0</kp>
+      <kd>1.0</kd>
+      <maxVel>0</maxVel>-->
+    </gazebo>
   </xacro:macro>
   <xacro:macro name="outer_finger_joint" params="prefix fingerprefix">
@@ -242,13 +249,15 @@
       </collision>
     </link>
-    <!--<gazebo reference="${prefix}${fingerprefix}_finger_tip">
-      <selfCollide>true</selfCollide>
-      <gravity>false</gravity>
-      <implicitSpringDamper>1</implicitSpringDamper>
-      <mu1>100000</mu1>
-      <mu2>100000</mu2>
-      <kp>100000000.0</kp>
-      <kd>1.0</kd>
-    </gazebo>-->
+    <gazebo reference="${prefix}${fingerprefix}_finger_tip">
+      <material>Gazebo/FlatBlack</material>
+      <!--<selfCollide>true</selfCollide>
+      <gravity>false</gravity>
+      <implicitSpringDamper>1</implicitSpringDamper>
+      <mu1>100000</mu1>
+      <mu2>100000</mu2>
+      <kp>100000000.0</kp>
+      <kd>1.0</kd>
+      <maxVel>0</maxVel>-->
+    </gazebo>
   </xacro:macro>
   <xacro:macro name="finger_tip_joint" params="prefix fingerprefix">

File: owr_description/urdf/gripper/robotiq_fts300.urdf.xacro (robot description, xacro)
@@ -45,4 +45,8 @@
         </joint>
         <link name="${prefix}fts_toolside"/>
+        <gazebo reference="${prefix}fts_robotside">
+            <selfCollide>true</selfCollide>
+            <material>Gazebo/Black</material>
+        </gazebo>
     </xacro:macro>
 </robot>

File: owr_description/urdf/owr.gazebo.xacro (robot description, xacro)
@@ -4,26 +4,34 @@
         <gazebo reference="${prefix}base_link">
             <selfCollide>true</selfCollide>
+            <material>Gazebo/Black</material>
         </gazebo>
         <gazebo reference="${prefix}BS_Link">
             <selfCollide>true</selfCollide>
+            <material>Gazebo/DarkGrey</material>
         </gazebo>
         <gazebo reference="${prefix}SE_Link">
             <selfCollide>true</selfCollide>
+            <material>Gazebo/Grey</material>
         </gazebo>
         <gazebo reference="${prefix}EW1_Link">
             <selfCollide>true</selfCollide>
+            <material>Gazebo/DarkGrey</material>
         </gazebo>
         <gazebo reference="${prefix}W1W2_Link">
             <selfCollide>true</selfCollide>
+            <material>Gazebo/Grey</material>
         </gazebo>
         <gazebo reference="${prefix}W2W3_Link">
             <selfCollide>true</selfCollide>
+            <material>Gazebo/DarkGrey</material>
         </gazebo>
         <gazebo reference="${prefix}W3EEF_Link">
             <selfCollide>true</selfCollide>
+            <material>Gazebo/Grey</material>
         </gazebo>
-        <gazebo reference="${prefix}EEF_Link">
+        <!--<gazebo reference="${prefix}EEF_Link">
             <selfCollide>true</selfCollide>
-        </gazebo>
+            <material>Gazebo/Red</material>
+        </gazebo>-->
     </xacro:macro>
 </robot>
